File: pcb/esp8266-led.brd (EAGLE design)
At the start: 45.7 x 45.7 mm, 26 parts

Commit message: Updated MOSFET dersistor values.
Parts:
- R5: value 10K -> 120R
- R6: value 10K -> 120K
Changed lines of the file:
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@@
 <attribute name="VALUE" x="9.144" y="10.795" size="1.27" layer="27" rot="R270"/>
 </element>
-<element name="R5" library="rcl" package="R0805" value="10K" x="36.322" y="25.4" smashed="yes" rot="MR180">
+<element name="R5" library="rcl" package="R0805" value="120R" x="36.322" y="25.4" smashed="yes" rot="MR180">
 <attribute name="NAME" x="38.354" y="24.765" size="1.27" layer="26" font="vector" ratio="15" rot="MR90"/>
 <attribute name="VALUE" x="35.687" y="27.94" size="1.27" layer="28" rot="MR180"/>
 </element>
-<element name="R6" library="rcl" package="R0805" value="10K" x="36.322" y="23.368" smashed="yes" rot="MR180">
+<element name="R6" library="rcl" package="R0805" value="120K" x="36.322" y="23.368" smashed="yes" rot="MR180">
 <attribute name="NAME" x="38.354" y="21.717" size="1.27" layer="26" font="vector" ratio="15" rot="MR90"/>
 <attribute name="VALUE" x="35.687" y="25.908" size="1.27" layer="28" rot="MR180"/>
